Commit message: change stl directory

File: nyangachi/urdf/macros.xacro (robot description, xacro)
@@ -9,7 +9,8 @@
             </inertial> -->
             <collision name="${name}_collision">
-                 <origin xyz="0 0 0" rpy="3.14 0 0"/>
+                <origin xyz="0 0 0" rpy="3.14 0 0"/>
               <geometry>
-                <box size="0.05 0.05 0.3"/>
+                <!-- <box size="0.05 0.05 0.3"/> -->
+                <mesh filename="stl/Forearm.stl" scale="1 1 1"/>
               </geometry>
             </collision>
@@ -35,5 +36,6 @@
                  <origin xyz="0 0 0" rpy="1.57 0 0"/>
               <geometry>
-                <box size="0.05 0.05 0.3"/>
+                <mesh filename="stl/Thigh.stl" scale="1 1 1"/>
+                <!-- <box size="0.05 0.05 0.3"/> -->
               </geometry>
             </collision>

Commit message: upload urdf file

File: nyangachi/urdf/macros.xacro (robot description, xacro)
@@ -1,5 +1,7 @@
 <?xml version="1.0"?>
-<robot>
-    <macro name="link_forearm" params="name">
+<robot xmlns:xacro="http://www.ros.org/wiki/xacro">
+    <!-- <xacro:include filename="$(find nyangachi)/urdf/materials.xacro" /> -->
+    <xacro:include filename="$(find nyangachi)/urdf/variables.xacro" />
+    <macro name="link_forearm" params="name origin_xyz">
         <link name="${name}">
             <!-- <inertial>
@@ -9,14 +11,16 @@
             </inertial> -->
             <collision name="${name}_collision">
-                <origin xyz="0 0 0" rpy="3.14 0 0"/>
+                <!-- <origin xyz="0 0 0" rpy="3.14 0 0"/> -->
+                <origin xyz="${origin_xyz}" rpy="0 0 0"/>
               <geometry>
-                <!-- <box size="0.05 0.05 0.3"/> -->
-                <mesh filename="stl/Forearm.stl" scale="1 1 1"/>
+                <box size="0.05 ${forearm_ylength} ${forearm_length}"/>
+                <!-- <mesh filename="~/simulation_ws/src/Nyangachi_Robot/stl/Forearm_ascii.stl" scale="1 1 1"/> -->
               </geometry>
             </collision>
             <visual name="${name}_visual">
-                <origin xyz="0 0 0" rpy="3.14 0 0"/>
+                <!-- <origin xyz="0 0 0" rpy="3.14 0 0"/> -->
+                <origin xyz="${origin_xyz}" rpy="0 0 0"/>
                 <geometry>
-                <box size="0.05 0.05 0.3"/>
+                <box size="${forearm_xlength} ${forearm_ylength} 0.3"/>
                 </geometry>
                 <material name="blue">
@@ -26,5 +30,5 @@
         </link>
     </macro>
-   <macro name="link_thigh" params="name">
+   <macro name="link_thigh" params="name origin_xyz">
         <link name="${name}">
             <!-- <inertial>
@@ -34,14 +38,16 @@
             </inertial> -->
             <collision name="${name}_collision">
-                 <origin xyz="0 0 0" rpy="1.57 0 0"/>
+                 <origin xyz="${origin_xyz}" rpy="0 0 0"/>
+                 <!-- <origin xyz="0 0 0" rpy="1.57 0 0"/> -->
               <geometry>
-                <mesh filename="stl/Thigh.stl" scale="1 1 1"/>
-                <!-- <box size="0.05 0.05 0.3"/> -->
+                <!-- <mesh filename="~/simulation_ws/src/Nyangachi_Robot/stl/Thigh_ascii.stl" scale="1 1 1"/> -->
+                <box size="${thigh_xlength} ${thigh_ylength} ${thigh_length}"/>
               </geometry>
             </collision>
             <visual name="${name}_visual">
-                <origin xyz="0 0 0" rpy="1.57 0 0"/>
+                <origin xyz="${origin_xyz}" rpy="0 0 0"/>
+                <!-- <origin xyz="0 0 0" rpy="1.57 0 0"/> -->
                 <geometry>
-                <box size="0.05 0.05 0.3"/>
+                <box size="${thigh_xlength} ${thigh_ylength} 0.3"/>
                 </geometry>
                 <material name="green">

File: nyangachi/urdf/main_nyang.xacro (robot description, xacro)
@@ -1,5 +1,6 @@
 <?xml version="1.0" ?>
 <robot name="nyangachi" xmlns:xacro="http://www.ros.org/wiki/xacro">
-  <xacro:include filename="$(find nyangachi)/urdf/materials.xacro" />
+  <!-- <xacro:include filename="$(find nyangachi)/urdf/materials.xacro" /> -->
+  <xacro:include filename="$(find nyangachi)/urdf/variables.xacro" />
   <!-- <xacro:include filename="$(find nyangachi)/urdf/m2wr.gazebo" /> -->
   <xacro:include filename="$(find nyangachi)/urdf/macros.xacro" />
@@ -51,19 +52,19 @@
     </visual>
   </link>
-    <xacro:joint_chassis_thigh name="joint_fr_thigh" child="link_fr_thigh" origin_xyz="0.3 0.15 0.04" />
-    <xacro:link_thigh name="link_fr_thigh" />
-    <!-- <xacro:joint_thigh_forearm name="joint_fr_forearm" child="link_fr_forearm" parent="link_fr_thigh" origin_xyz="0 0 0.3" />
-    <xacro:link_forearm name="link_fr_forearm" /> -->
-    <xacro:joint_chassis_thigh name="joint_fl_thigh" child="link_fl_thigh" origin_xyz="0.3 -0.15 0.04" />
-    <xacro:link_thigh name="link_fl_thigh" />
-    <!-- <xacro:joint_thigh_forearm name="joint_fl_forearm" child="link_fl_forearm" parent="link_fl_thigh" origin_xyz="0 0 0.3" />
-    <xacro:link_forearm name="link_fl_forearm" /> -->
-    <xacro:joint_chassis_thigh name="joint_br_thigh" child="link_br_thigh" origin_xyz="-0.3 -0.15 0.04" />
-    <xacro:link_thigh name="link_br_thigh" />
-    <!-- <xacro:joint_thigh_forearm name="joint_br_forearm" child="link_br_forearm" parent="link_br_thigh" origin_xyz="0 0 0.3" />
-    <xacro:link_forearm name="link_br_forearm" /> -->
-    <xacro:joint_chassis_thigh name="joint_bl_thigh" child="link_bl_thigh" origin_xyz="-0.3 -0.15 0.04" />
-    <xacro:link_thigh name="link_bl_thigh" />
-    <!-- <xacro:joint_thigh_forearm name="joint_bl_forearm" child="link_bl_forearm" parent="link_bl_thigh" origin_xyz="0 0 0.3" />
-    <xacro:link_forearm name="link_bl_forearm" /> -->
+    <xacro:joint_chassis_thigh name="joint_fr_thigh" child="link_fr_thigh" origin_xyz="${0.25-thigh_xlength/2} ${0.15+thigh_ylength/2} 0" />
+    <xacro:link_thigh name="link_fr_thigh" origin_xyz = "0 0 ${-thigh_length/2}" />
+    <xacro:joint_thigh_forearm name="joint_fr_forearm" child="link_fr_forearm" parent="link_fr_thigh" origin_xyz="0 ${forearm_ylength} ${-thigh_length}" />
+    <xacro:link_forearm name="link_fr_forearm" origin_xyz = "0 0 ${-forearm_length/2}" />
+    <xacro:joint_chassis_thigh name="joint_fl_thigh" child="link_fl_thigh" origin_xyz="${0.25-thigh_xlength/2} -${0.15+thigh_ylength/2} 0" />
+    <xacro:link_thigh name="link_fl_thigh" origin_xyz = "0 0 ${-thigh_length/2}"/>
+    <xacro:joint_thigh_forearm name="joint_fl_forearm" child="link_fl_forearm" parent="link_fl_thigh" origin_xyz="0 -${forearm_ylength} ${-thigh_length}" />
+    <xacro:link_forearm name="link_fl_forearm" origin_xyz = "0 0 ${-forearm_length/2}"/>
+    <xacro:joint_chassis_thigh name="joint_br_thigh" child="link_br_thigh" origin_xyz="-${0.25-thigh_xlength/2} ${0.15+thigh_ylength/2} 0.0" />
+    <xacro:link_thigh name="link_br_thigh" origin_xyz = "0 0 ${-thigh_length/2}"/>
+    <xacro:joint_thigh_forearm name="joint_br_forearm" child="link_br_forearm" parent="link_br_thigh" origin_xyz="0 ${forearm_ylength} ${-thigh_length}" />
+    <xacro:link_forearm name="link_br_forearm" origin_xyz = "0 0 ${-forearm_length/2}"/>
+    <xacro:joint_chassis_thigh name="joint_bl_thigh" child="link_bl_thigh" origin_xyz="-${0.25-thigh_xlength/2} -${0.15+thigh_ylength/2} 0.0" />
+    <xacro:link_thigh name="link_bl_thigh" origin_xyz = "0 0 ${-thigh_length/2}"/>
+    <xacro:joint_thigh_forearm name="joint_bl_forearm" child="link_bl_forearm" parent="link_bl_thigh" origin_xyz="0 -${forearm_ylength} ${-thigh_length}" />
+    <xacro:link_forearm name="link_bl_forearm" origin_xyz = "0 0 ${-forearm_length/2}"/>
 </robot>
